File: PCB-Case/Psycho-Ducker-case/frontplate/Psycho-Ducker-case.kicad_pcb (KiCad board)
At the start: 2 copper layers, 310.6 x 124.2 mm, 0 parts

Commit message: feat: added mounting holes
Routing:
- added copper zone on B.Cu, net (none)
- added copper zone on F.Cu, net (none)
Other:
- outline, holes or cut-outs redrawn
- board text removed: "scale: 0,0395036"
