File: PCB-Case/Psycho-Ducker-case/backplate/backplate.kicad_pcb (KiCad board)
At the start: 2 copper layers, 310 x 124 mm, 2 parts

Commit message: fix: removed useless folder
Parts:
- added G***: LOGO, LOGO, F.Cu at (218.0, 140.0)
Routing:
- net (no net): track 8970.7 -> 8834.6 mm
Other:
- board text added: "PSYCHO DUCKER BOTTOM PLATE V1.0 by Angelo Perotti"
- board text removed: "PSYCHO DUCKER BOTTOM PLATE V1.0"
