File: KiCad/psycho_ducker.kicad_sch (KiCad schematic)
At the start: 187 parts, among them J1 USB_C, SW1 SW_Push, U1 STM32F072CBT6, U3 XC6206, U4 USBLC6-2SC6

Commit message: fix: c7 footprint, jlc code repetition, shrek typo and added duck
Parts:
- C7: footprint ScottoKeebs_Components:Diode_SOD-123 -> ScottoKeebs_Components:Capacitor_0402
Other:
- note removed: "LEDs"
Changed lines of the file:
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@@
 	)
 	(rectangle
-		(start 25.4 25.4)
-		(end 114.3 101.6)
-		(stroke
-			(width 0)
-			(type default)
-		)
-		(fill
-			(type none)
-		)
-	)
-	(rectangle
 		(start 124.46 215.9)
 		(end 259.08 281.94)
@@
 		)
 	)
-	(rectangle
-		(start 105.41 93.98)
-		(end 105.41 93.98)
-		(stroke
-			(width 0)
-			(type default)
-		)
-		(fill
-			(type none)
-		)
-	)
 	(text_box "Hold when plugging in to enter bootloader mode."
 		(exclude_from_sim no)
@@
 		)
 	)
-	(text "LEDs\n"
-		(exclude_from_sim no)
-		(at 27.432 24.13 0)
-		(effects
-			(font
-				(size 1.27 1.27)
-			)
-		)
-	)
 	(text "Matrix"
 		(exclude_from_sim no)
@@
 			)
 		)
-		(property "Footprint" "ScottoKeebs_Components:Diode_SOD-123"
+		(property "Footprint" "ScottoKeebs_Components:Capacitor_0402"
 			(at 27.94 175.26 0)
 			(effects
@@
 	)
 	(symbol
-		(lib_id "power:+3.3V")
-		(at 38.1 38.1 0)
-		(unit 1)
-		(exclude_from_sim no)
-		(in_bom yes)
-		(on_board yes)
-		(dnp no)
-		(property "Reference" "#PWR01"
-			(at 38.1 41.91 0)
-			(effects
-				(font
-					(size 1.27 1.27)
-				)
-				(hide yes)
-			)
-		)
-		(property "Value" "+3.3V"
-			(at 37.846 34.29 0)
-			(effects
-				(font
-					(size 1.27 1.27)
-				)
-			)
-		)
-		(property "Footprint" ""
-			(at 38.1 38.1 0)
-			(effects
-				(font
-					(size 1.27 1.27)
-				)
-				(hide yes)
-			)
-		)
-		(property "Datasheet" ""
-			(at 38.1 38.1 0)
-			(effects
-				(font
-					(size 1.27 1.27)
-				)
-				(hide yes)
-			)
-		)
-		(property "Description" "Power symbol creates a global label with name \"+3.3V\""
-			(at 38.1 38.1 0)
-			(effects
-				(font
-					(size 1.27 1.27)
-				)
-				(hide yes)
-			)
-		)
-		(pin "1"
-		)
-		(instances
-			(project "psycho_ducker"
-				(path "/92054fa3-5ad0-458e-bd73-acbcf8d11243"
-					(reference "#PWR01")
-					(unit 1)
-				)
-			)
-		)
-	)
-	(symbol
 		(lib_id "scottokeebs:Placeholder_Diode")
 		(at 207.01 71.12 90)
@@
 					(unit 1)
 				)
-			)
-		)
-	)
-	(symbol
-		(lib_id "power:GND")
-		(at 38.1 76.2 0)
-		(unit 1)
-		(exclude_from_sim no)
-		(in_bom yes)
-		(on_board yes)
-		(dnp no)
-		(property "Reference" "#PWR03"
-			(at 38.1 82.55 0)
-			(effects
-				(font
-					(size 1.27 1.27)
-				)
-				(hide yes)
-			)
-		)
-		(property "Value" "GND"
-			(at 37.846 80.264 0)
-			(effects
-				(font
-					(size 1.27 1.27)
-				)
-			)
-		)
-		(property "Footprint" ""
-			(at 38.1 76.2 0)
-			(effects
-				(font
-					(size 1.27 1.27)
-				)
-				(hide yes)
-			)
-		)
-		(property "Datasheet" ""
-			(at 38.1 76.2 0)
-			(effects
-				(font
-					(size 1.27 1.27)
-				)
-				(hide yes)
-			)
-		)
-		(property "Description" "Power symbol creates a global label with name \"GND\" , ground"
-			(at 38.1 76.2 0)
-			(effects
-				(font
-					(size 1.27 1.27)
-				)
-				(hide yes)
-			)
-		)
-		(pin "1"
-		)
-		(instances
-			(project "psycho_ducker"
-				(path "/92054fa3-5ad0-458e-bd73-acbcf8d11243"
-					(reference "#PWR03")
-					(unit 1)
-				)

Commit message: fix: removed holes from schematic
Parts:
- removed H1, H2, H3, H4, H5, H6, H7: Mounting_Hole, symbol ScottoKeebs:Placeholder_Mounting_Hole
