File: KiCad/psycho_ducker.kicad_sch (KiCad schematic)
At the start: 180 parts, among them J1 USB_C, SW1 SW_Push, U1 STM32F072CBT6, U3 XC6206, U4 USBLC6-2SC6

Commit message: feat: added WS2812B to the pcb
Parts:
- added C1, C2, C3, C4, C5, C57, C6: 100n, Capacitor_SMD:C_0603_1608Metric, symbol Device:C
- added C19: 100nF, Capacitor_SMD:C_0603_1608Metric, symbol Device:C_Small
- added D81, D82, D83, D84, D85, D86, D87: WS2812B, LED_SMD:LED_WS2812B_PLCC4_5.0x5.0mm_P3.2mm, symbol LED:WS2812B
- added JP1: SolderJumper_2_Open, Jumper:SolderJumper-2_P1.3mm_Open_RoundedPad1.0x1.5mm, symbol Jumper:SolderJumper_2_Open
- added R4: 330, Resistor_SMD:R_0603_1608Metric, symbol Device:R
- added U2: 74AHCT1G125, Package_TO_SOT_SMD:SOT-23-5_HandSoldering, symbol 74xGxx:74AHCT1G125
Connections:
- net +5V: now also C1.1, C19.2, C2.1, C3.1, C4.1, C5.1, C57.1, C6.1, D81.1 (VDD), D82.1 (VDD), D83.1 (VDD), D84.1 (VDD), D85.1 (VDD), D86.1 (VDD), D87.1 (VDD), U2.5 (VCC)
- net F0: now also JP1.2 (B)
- net GND: now also C1.2, C19.1, C2.2, C3.2, C4.2, C5.2, C57.2, C6.2, D81.3 (VSS), D82.3 (VSS), D83.3 (VSS), D84.3 (VSS), D85.3 (VSS), D86.3 (VSS), D87.3 (VSS), JP1.1 (A), U2.1, U2.3 (GND)
- net LED_OUT: now reaches U1.16 (PA6)
- net LED_OUT: now also U2.2
- new net: D83.2 (DOUT), D84.4 (DIN)
- new net: D82.2 (DOUT), D83.4 (DIN)
- new net: D84.2 (DOUT), D85.4 (DIN)
- new net: R4.1, U2.4
- new net: D81.2 (DOUT), D82.4 (DIN)
- new net: D81.4 (DIN), R4.2
- new net: D86.2 (DOUT), D87.4 (DIN)
- new net: D85.2 (DOUT), D86.4 (DIN)
Other:
- note added: "in"
- note added: "out"
- note removed: "Mounting Holes"
- moved on the sheet: D1, D10, D11, D12, D13, D14, D15, D16, D17, D18, D19, D2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
