File: KiCad/psycho_ducker.kicad_pcb (KiCad board)
At the start: 2 copper layers, 310.6 x 124.3 mm, 187 parts, among them J1 USB_C, SW1 SW_Push, U1 STM32F072CBT6, U3 XC6206, U4 USBLC6-2SC6

Commit message: fix: removed MCU and various IC for a start=over routing journey
Parts:
- removed C10, C11, C13, C16, C7: 100nF, ScottoKeebs_Components:Capacitor_0402
- removed C12, C17: 4.7uF, ScottoKeebs_Components:Capacitor_0402
- removed C14: 10nF, ScottoKeebs_Components:Capacitor_0402
- removed C15, C8, C9: 1uF, ScottoKeebs_Components:Capacitor_0402
- removed F1: 500mA, ScottoKeebs_Components:Fuse_0603
- removed R1: 10k, Resistor_SMD:R_0402_1005Metric
- removed R2, R3: 5.1k, Resistor_SMD:R_0402_1005Metric
- removed SW1: SW_Push, ScottoKeebs_Components:Button_TL3342
- removed U1: STM32F072CBT6, ScottoKeebs_Components:Package_LQFP-48_7x7mm_P0.5
- removed U3: XC6206, ScottoKeebs_Components:Voltage_SOT-23
- removed U4: USBLC6-2SC6, ScottoKeebs_Components:ESD_SOT-23-6
Routing:
- net /B9: track 462.5 -> 92.1 mm, vias 5 -> 0
- net /B6: track 406.8 -> 112.9 mm, vias 1 -> 0
- net /B7: track 390.1 -> 120.3 mm, vias 1 -> 0
- net /B8: track 377.9 -> 122.0 mm, vias 1 -> 0
- net /B10: track 330.0 -> 94.2 mm, vias 1 -> 0
- net /B11: track 342.8 -> 117.7 mm, vias 1 -> 0
- net /B12: track 279.3 -> 99.5 mm, vias 1 -> 0
- net /B13: track 272.5 -> 97.6 mm, vias 1 -> 0
- net /B14: track 268.9 -> 120.8 mm, vias 1 -> 0
- net GND: track 147.2 -> 0.00 mm, vias 3 -> 0
- net /B5: track 460.1 -> 314.7 mm, vias 12 -> 9
- net /B4: track 428.7 -> 291.7 mm, vias 14 -> 13
- net /B15: track 225.3 -> 97.1 mm, vias 1 -> 0
- net +3.3V: track 125.6 -> 0.00 mm, vias 1 -> 0
- net /A0: track 223.6 -> 119.7 mm, vias 1 -> 0
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
Commit message: feat: updated routing
Parts:
- added C10: 100nF, ScottoKeebs_Components:Capacitor_0402, F.Cu at (561.2, 223.7)
- added C11: 100nF, ScottoKeebs_Components:Capacitor_0402, F.Cu at (568.1, 233.4)
- added C12: 4.7uF, ScottoKeebs_Components:Capacitor_0402, F.Cu at (568.1, 234.4)
- added C13: 100nF, ScottoKeebs_Components:Capacitor_0402, F.Cu at (562.9, 222.1)
- added C14: 10nF, ScottoKeebs_Components:Capacitor_0402, F.Cu at (559.3, 228.9)
- added C15: 1uF, ScottoKeebs_Components:Capacitor_0402, F.Cu at (558.3, 228.9)
- added C16: 100nF, ScottoKeebs_Components:Capacitor_0402, F.Cu at (571.1, 225.3)
- added C17: 4.7uF, ScottoKeebs_Components:Capacitor_0402, F.Cu at (572.1, 225.3)
- added C7: 100nF, ScottoKeebs_Components:Capacitor_0402, F.Cu at (558.8, 227.5)
- added C8: 1uF, ScottoKeebs_Components:Capacitor_0402, F.Cu at (579.5, 220.3)
- added C9: 1uF, ScottoKeebs_Components:Capacitor_0402, F.Cu at (580.2, 225.2)
- added F1: 500mA, ScottoKeebs_Components:Fuse_0603, F.Cu at (577.8, 219.3)
- added R1: 10k, Resistor_SMD:R_0402_1005Metric, F.Cu at (582.4, 225.2)
- added R2: 5.1k, Resistor_SMD:R_0402_1005Metric, F.Cu at (574.0, 218.8)
- added R3: 5.1k, Resistor_SMD:R_0402_1005Metric, F.Cu at (576.1, 218.7)
- added SW1: SW_Push, ScottoKeebs_Components:Button_TL3342, F.Cu at (579.9, 230.0)
- added U1: STM32F072CBT6, ScottoKeebs_Components:Package_LQFP-48_7x7mm_P0.5, F.Cu at (565.5, 227.8)
- added U3: XC6206, ScottoKeebs_Components:Voltage_SOT-23, F.Cu at (580.1, 222.8)
- added U4: USBLC6-2SC6, ScottoKeebs_Components:ESD_SOT-23-6, F.Cu at (575.3, 222.8)
Routing:
- net /B6: track 112.9 -> 412.4 mm, vias 0 -> 1
- net /B7: track 120.3 -> 394.9 mm, vias 0 -> 1
- net /B8: track 122.0 -> 376.7 mm, vias 0 -> 1
- net /B9: track 92.1 -> 326.8 mm, vias 0 -> 1
- net /B13: track 97.6 -> 255.8 mm, vias 0 -> 3
- net /B12: track 99.5 -> 253.7 mm, vias 0 -> 2
- net /B14: track 120.8 -> 248.7 mm, vias 0 -> 3
- net /B11: track 117.7 -> 241.7 mm, vias 0 -> 2
- net /B5: track 314.7 -> 436.5 mm, vias 9 -> 12
- net /B15: track 97.1 -> 205.6 mm, vias 0 -> 3
- net /B4: track 291.7 -> 397.7 mm, vias 13 -> 16
- net GND: track 0.00 -> 88.7 mm
- net /A0: track 119.7 -> 208.4 mm, vias 0 -> 1
- net /A1: track 133.4 -> 211.1 mm, vias 0 -> 1
- net /B3: track 321.8 -> 398.3 mm, vias 14 -> 17
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