File: PCB-Case/FR-4_Case/frontplate/Psycho-Ducker-case.kicad_pcb (KiCad board)
At the start: 2 copper layers, 310.6 x 124.2 mm, 0 parts

Commit message: fix: added border for plate mount
Parts:
- added G***: LOGO, LOGO, F.Cu at (358.7, 80.3)
Routing:
- net (no net): track 8970.7 -> 0.00 mm
Other:
- board size 310.6 x 124.2 mm -> 310.6 x 134.3 mm
- board text added: "*Duck noise intensifies*"
- board text added: "BA DUM TSSS"
